File: Vi-Fi.kicad_sch (KiCad schematic)
At the start: 19 parts, among them J1 4P4C, SW1 SW_SPST, U1 ESP-WROOM-02, U2 CS48520S, U3 MP1469

Commit message: Board Layout Started
Parts:
- removed D1: LED, symbol Device:LED
- removed R10, R8: 10K, symbol Device:R
- removed SW1: SW_SPST, symbol Switch:SW_SPST
- added C2: 0.1u, Capacitor_SMD:C_0603_1608Metric, symbol Device:C
- added SW2: C2681568, Vi-Fi:C2681568, symbol Vi-Fi_Parts:C2681568
- C1, C2A1: footprint (none) -> Capacitor_SMD:C_0805_2012Metric
- C1A1, C3, C4: footprint (none) -> Capacitor_SMD:C_0603_1608Metric
- J1: footprint (none) -> Connector_RJ:RJ9_Evercom_5301-440xxx_Horizontal
- L1: value 6.5u -> 6.8u; footprint (none) -> Vi-Fi:L_CD73
- R1, R2, R5, R7, R9: footprint (none) -> Resistor_SMD:R_0603_1608Metric
- U1: value ESP-WROOM-02 -> ESP-WROOM-02D-N4
- U2: footprint (none) -> Package_SO:SOIC-8_3.9x4.9mm_P1.27mm
- U3: footprint (none) -> Package_TO_SOT_SMD:TSOT-23-6
Connections:
- net +3V3: now also C2.1, SW2.3 (C)
- net GND: now also C2.2, SW2.1 (A), SW2.4 (GND)
- net at U1.8 (IO0): now also SW2.2 (B)
Other:
- moved on the sheet: C2A1
